File: FPGA-Power.sch (KiCad schematic (older format))
At the start: 1 part, among them U1 10CL040_F484

Commit message: Made progress woth power
Signed-off-by: Jan Mart Liewes <Eldalote.Electronics@gmail.com>
Parts:
- renumbered U1 to U1201
Changed lines of the file:
@@
 $Descr A4 11693 8268
 encoding utf-8
-Sheet 11 12
+Sheet 11 15
 Title ""
 Date ""
@@
 $EndDescr
 $Comp
-L Cyclone10LP_040:10CL040_F484 U1
+L Cyclone10LP_040:10CL040_F484 U1201
 U 12 1 5F5290CD
 P 9350 750
-F 0 "U1" H 10427 -2075 35  0000 L CNN
+F 0 "U1201" H 10427 -2075 35  0000 L CNN
 F 1 "10CL040_F484" H 10400 -5175 35  0001 L CNN
 F 2 "SamacSys_Parts:BGA484C100P22X22_2300X2300X200" H 10400 -5220 35  0001 L CNN
@@
 $EndComp
 $Comp
-L Cyclone10LP_040:10CL040_F484 U1
+L Cyclone10LP_040:10CL040_F484 U1201
 U 13 1 5F537C92
 P 6450 5500
-F 0 "U1" H 7527 5188 35  0000 L CNN
+F 0 "U1201" H 7527 5188 35  0000 L CNN
 F 1 "10CL040_F484" H 7500 -425 35  0001 L CNN
 F 2 "SamacSys_Parts:BGA484C100P22X22_2300X2300X200" H 7500 -470 35  0001 L CNN
@@
 $EndComp
 $Comp
-L Cyclone10LP_040:10CL040_F484 U1
+L Cyclone10LP_040:10CL040_F484 U1201
 U 1 1 5F54588B
 P 2450 700
-F 0 "U1" H 3527 -2312 35  0000 L CNN
+F 0 "U1201" H 3527 -2312 35  0000 L CNN
 F 1 "10CL040_F484" H 3500 -5225 35  0001 L CNN
 F 2 "SamacSys_Parts:BGA484C100P22X22_2300X2300X200" H 3500 -5270 35  0001 L CNN
