File: FPGA1.sch (KiCad schematic (older format))
At the start: 1 part, among them U1 10CL040_F484

Commit message: Made progress woth power
Signed-off-by: Jan Mart Liewes <Eldalote.Electronics@gmail.com>
Parts:
- renumbered U1 to U1201
Changed lines of the file:
@@
 $Descr A4 11693 8268
 encoding utf-8
-Sheet 8 12
+Sheet 8 15
 Title ""
 Date ""
@@
 $EndDescr
 $Comp
-L Cyclone10LP_040:10CL040_F484 U1
+L Cyclone10LP_040:10CL040_F484 U1201
 U 2 1 5F48E945
 P 2750 1200
-F 0 "U1" H 3827 100 35  0000 L CNN
+F 0 "U1201" H 3827 100 35  0000 L CNN
 F 1 "10CL040_F484" H 3800 -4725 35  0001 L CNN
 F 2 "SamacSys_Parts:BGA484C100P22X22_2300X2300X200" H 3800 -4770 35  0001 L CNN
@@
 $EndComp
 $Comp
-L Cyclone10LP_040:10CL040_F484 U1
+L Cyclone10LP_040:10CL040_F484 U1201
 U 3 1 5F4AE0F4
 P 6150 1200
-F 0 "U1" H 7227 -425 35  0000 L CNN
+F 0 "U1201" H 7227 -425 35  0000 L CNN
 F 1 "10CL040_F484" H 7200 -4725 35  0001 L CNN
 F 2 "SamacSys_Parts:BGA484C100P22X22_2300X2300X200" H 7200 -4770 35  0001 L CNN
@@
 $EndComp
 $Comp
-L Cyclone10LP_040:10CL040_F484 U1
+L Cyclone10LP_040:10CL040_F484 U1201
 U 4 1 5F4BF162
 P 9650 1300
-F 0 "U1" H 10802 -250 35  0000 L CNN
+F 0 "U1201" H 10802 -250 35  0000 L CNN
 F 1 "10CL040_F484" H 10700 -4625 35  0001 L CNN
 F 2 "SamacSys_Parts:BGA484C100P22X22_2300X2300X200" H 10700 -4670 35  0001 L CNN
