File: FPGA2.sch (KiCad schematic (older format))
At the start: 1 part, among them U1 10CL040_F484

Commit message: Made progress woth power
Signed-off-by: Jan Mart Liewes <Eldalote.Electronics@gmail.com>
Parts:
- renumbered U1 to U1201
Changed lines of the file:
@@
 $Descr A4 11693 8268
 encoding utf-8
-Sheet 9 12
+Sheet 9 15
 Title ""
 Date ""
@@
 $EndDescr
 $Comp
-L Cyclone10LP_040:10CL040_F484 U1
+L Cyclone10LP_040:10CL040_F484 U1201
 U 5 1 5F4CDD3F
 P 2200 1650
-F 0 "U1" H 3351 138 35  0000 L CNN
+F 0 "U1201" H 3351 138 35  0000 L CNN
 F 1 "10CL040_F484" H 3250 -4275 35  0001 L CNN
 F 2 "SamacSys_Parts:BGA484C100P22X22_2300X2300X200" H 3250 -4320 35  0001 L CNN
@@
 $EndComp
 $Comp
-L Cyclone10LP_040:10CL040_F484 U1
+L Cyclone10LP_040:10CL040_F484 U1201
 U 6 1 5F4D5123
 P 4900 1600
-F 0 "U1" H 5977 125 35  0000 L CNN
+F 0 "U1201" H 5977 125 35  0000 L CNN
 F 1 "10CL040_F484" H 5950 -4325 35  0001 L CNN
 F 2 "SamacSys_Parts:BGA484C100P22X22_2300X2300X200" H 5950 -4370 35  0001 L CNN
@@
 $EndComp
 $Comp
-L Cyclone10LP_040:10CL040_F484 U1
+L Cyclone10LP_040:10CL040_F484 U1201
 U 7 1 5F4E58F6
 P 7850 1850
-F 0 "U1" H 8927 638 35  0000 L CNN
+F 0 "U1201" H 8927 638 35  0000 L CNN
 F 1 "10CL040_F484" H 8900 -4075 35  0001 L CNN
 F 2 "SamacSys_Parts:BGA484C100P22X22_2300X2300X200" H 8900 -4120 35  0001 L CNN
