File: FPGA3.sch (KiCad schematic (older format))
At the start: 1 part, among them U1 10CL040_F484

Commit message: Made progress woth power
Signed-off-by: Jan Mart Liewes <Eldalote.Electronics@gmail.com>
Parts:
- renumbered U1 to U1201
Changed lines of the file:
@@
 $Descr A4 11693 8268
 encoding utf-8
-Sheet 10 12
+Sheet 10 15
 Title ""
 Date ""
@@
 $EndDescr
 $Comp
-L Cyclone10LP_040:10CL040_F484 U1
+L Cyclone10LP_040:10CL040_F484 U1201
 U 8 1 5F4F44FA
 P 2600 1500
-F 0 "U1" H 3752 -87 35  0000 L CNN
+F 0 "U1201" H 3752 -87 35  0000 L CNN
 F 1 "10CL040_F484" H 3650 -4425 35  0001 L CNN
 F 2 "SamacSys_Parts:BGA484C100P22X22_2300X2300X200" H 3650 -4470 35  0001 L CNN
@@
 $EndComp
 $Comp
-L Cyclone10LP_040:10CL040_F484 U1
+L Cyclone10LP_040:10CL040_F484 U1201
 U 9 1 5F5011A2
 P 5800 1700
-F 0 "U1" H 6877 338 35  0000 L CNN
+F 0 "U1201" H 6877 338 35  0000 L CNN
 F 1 "10CL040_F484" H 6850 -4225 35  0001 L CNN
 F 2 "SamacSys_Parts:BGA484C100P22X22_2300X2300X200" H 6850 -4270 35  0001 L CNN
@@
 $EndComp
 $Comp
-L Cyclone10LP_040:10CL040_F484 U1
+L Cyclone10LP_040:10CL040_F484 U1201
 U 10 1 5F50A9B4
 P 9150 1450
-F 0 "U1" H 10377 -587 35  0000 L CNN
+F 0 "U1201" H 10377 -587 35  0000 L CNN
 F 1 "10CL040_F484" H 10200 -4475 35  0001 L CNN
 F 2 "SamacSys_Parts:BGA484C100P22X22_2300X2300X200" H 10200 -4520 35  0001 L CNN
@@
 $EndComp
 $Comp
-L Cyclone10LP_040:10CL040_F484 U1
+L Cyclone10LP_040:10CL040_F484 U1201
 U 11 1 5F515CFB
 P 5050 4850
-F 0 "U1" H 6352 3600 35  0000 L CNN
+F 0 "U1201" H 6352 3600 35  0000 L CNN
 F 1 "10CL040_F484" H 6100 -1075 35  0001 L CNN
 F 2 "SamacSys_Parts:BGA484C100P22X22_2300X2300X200" H 6100 -1120 35  0001 L CNN
