File: GPIO.sch (KiCad schematic (older format))
At the start: 5 parts, among them J701 Conn_02x10, J702 Conn_02x07, J703 Conn_02x10, J704 Conn_02x04, J705 Conn_02x05

Commit message: Made progress woth power
Signed-off-by: Jan Mart Liewes <Eldalote.Electronics@gmail.com>
Parts:
- renumbered J701 to J1001, J702 to J1002, J703 to J1003, J704 to J1004, J705 to J1005
Changed lines of the file:
@@
 $Descr A4 11693 8268
 encoding utf-8
-Sheet 7 12
+Sheet 7 15
 Title ""
 Date ""
@@
 P 1650 1500
 AR Path="/5F439C11/5F5C3855" Ref="J?"  Part="1"
-AR Path="/5F439C11/5F5C1DDB/5F5C3855" Ref="J701"  Part="1"
-F 0 "J701" H 1700 2117 50  0000 C CNN
+AR Path="/5F439C11/5F5C1DDB/5F5C3855" Ref="J1001"  Part="1"
+F 0 "J1001" H 1700 2117 50  0000 C CNN
 F 1 "Conn_02x10" H 1700 2050 50  0000 C CNN
 F 2 "Connector_PinHeader_2.54mm:PinHeader_2x10_P2.54mm_Vertical" H 1650 1500 50  0001 C CNN
@@
 P 5450 1500
 AR Path="/5F439C11/5F5C385B" Ref="J?"  Part="1"
-AR Path="/5F439C11/5F5C1DDB/5F5C385B" Ref="J703"  Part="1"
-F 0 "J703" H 5500 2117 50  0000 C CNN
+AR Path="/5F439C11/5F5C1DDB/5F5C385B" Ref="J1003"  Part="1"
+F 0 "J1003" H 5500 2117 50  0000 C CNN
 F 1 "Conn_02x10" H 5500 2026 50  0000 C CNN
 F 2 "Connector_PinHeader_2.54mm:PinHeader_2x10_P2.54mm_Vertical" H 5450 1500 50  0001 C CNN
@@
 $EndComp
 $Comp
-L Connector_Generic:Conn_02x07_Odd_Even J702
+L Connector_Generic:Conn_02x07_Odd_Even J1002
 U 1 1 5F5C7DF5
 P 1950 5900
-F 0 "J702" H 2000 6417 50  0000 C CNN
+F 0 "J1002" H 2000 6417 50  0000 C CNN
 F 1 "Conn_02x07" H 2000 6326 50  0000 C CNN
 F 2 "Connector_PinHeader_2.54mm:PinHeader_2x07_P2.54mm_Vertical" H 1950 5900 50  0001 C CNN
@@
 $EndComp
 $Comp
-L Connector_Generic:Conn_02x04_Odd_Even J704
+L Connector_Generic:Conn_02x04_Odd_Even J1004
 U 1 1 5F5C919C
 P 5500 5750
-F 0 "J704" H 5550 6067 50  0000 C CNN
+F 0 "J1004" H 5550 6067 50  0000 C CNN
 F 1 "Conn_02x04" H 5550 5976 50  0000 C CNN
 F 2 "Connector_PinHeader_2.54mm:PinHeader_2x04_P2.54mm_Vertical" H 5500 5750 50  0001 C CNN
@@
 $EndComp
 $Comp
-L Connector_Generic:Conn_02x05_Odd_Even J705
+L Connector_Generic:Conn_02x05_Odd_Even J1005
 U 1 1 5F5CA1BC
 P 8950 3550
-F 0 "J705" H 9000 3967 50  0000 C CNN
+F 0 "J1005" H 9000 3967 50  0000 C CNN
 F 1 "Conn_02x05" H 9000 3876 50  0000 C CNN
 F 2 "Connector_PinHeader_2.54mm:PinHeader_2x05_P2.54mm_Vertical" H 8950 3550 50  0001 C CNN
@@
 $EndComp
 $Comp
-L power:+3.3V #PWR0103
+L power:+3.3V #PWR01001
 U 1 1 5F5D0685
 P 1350 1100
-F 0 "#PWR0103" H 1350 950 50  0001 C CNN
+F 0 "#PWR01001" H 1350 950 50  0001 C CNN
 F 1 "+3.3V" H 1365 1273 50  0000 C CNN
 F 2 "" H 1350 1100 50  0001 C CNN
@@
 $EndComp
 $Comp
-L power:GND #PWR0104
+L power:GND #PWR01002
 U 1 1 5F5D1394
 P 1350 2000
-F 0 "#PWR0104" H 1350 1750 50  0001 C CNN
+F 0 "#PWR01002" H 1350 1750 50  0001 C CNN
 F 1 "GND" H 1355 1827 50  0000 C CNN
 F 2 "" H 1350 2000 50  0001 C CNN
@@
 $EndComp
 $Comp
-L power:GND #PWR0105
+L power:GND #PWR01006
 U 1 1 5F5D1A60
 P 2050 2000
-F 0 "#PWR0105" H 2050 1750 50  0001 C CNN
+F 0 "#PWR01006" H 2050 1750 50  0001 C CNN
 F 1 "GND" H 2055 1827 50  0000 C CNN
 F 2 "" H 2050 2000 50  0001 C CNN
@@
 $EndComp
 $Comp
-L power:+3.3V #PWR0106
+L power:+3.3V #PWR01005
 U 1 1 5F5D2E37
 P 2050 1100
-F 0 "#PWR0106" H 2050 950 50  0001 C CNN
+F 0 "#PWR01005" H 2050 950 50  0001 C CNN
 F 1 "+3.3V" H 2065 1273 50  0000 C CNN
 F 2 "" H 2050 1100 50  0001 C CNN
@@
 	1350 1100 1450 1100
 $Comp
-L power:+3.3V #PWR0107
+L power:+3.3V #PWR01009
 U 1 1 5F5D4E37
 P 5150 1100
-F 0 "#PWR0107" H 5150 950 50  0001 C CNN
+F 0 "#PWR01009" H 5150 950 50  0001 C CNN
 F 1 "+3.3V" H 5165 1273 50  0000 C CNN
 F 2 "" H 5150 1100 50  0001 C CNN
@@
 $EndComp
 $Comp
-L power:+3.3V #PWR0108
+L power:+3.3V #PWR01013
 U 1 1 5F5D53FF
 P 5850 1100
-F 0 "#PWR0108" H 5850 950 50  0001 C CNN
+F 0 "#PWR01013" H 5850 950 50  0001 C CNN
 F 1 "+3.3V" H 5865 1273 50  0000 C CNN
 F 2 "" H 5850 1100 50  0001 C CNN
@@
 $EndComp
 $Comp
-L power:GND #PWR0109
+L power:GND #PWR01010
 U 1 1 5F5D55FF
 P 5150 2000
-F 0 "#PWR0109" H 5150 1750 50  0001 C CNN
+F 0 "#PWR01010" H 5150 1750 50  0001 C CNN
 F 1 "GND" H 5155 1827 50  0000 C CNN
 F 2 "" H 5150 2000 50  0001 C CNN
@@
 $EndComp
 $Comp
-L power:GND #PWR0110
+L power:GND #PWR01014
 U 1 1 5F5D58BC
 P 5850 2000
-F 0 "#PWR0110" H 5850 1750 50  0001 C CNN
+F 0 "#PWR01014" H 5850 1750 50  0001 C CNN
 F 1 "GND" H 5855 1827 50  0000 C CNN
 F 2 "" H 5850 2000 50  0001 C CNN
@@
 	5850 2000 5750 2000
 $Comp
-L power:GND #PWR0111
+L power:GND #PWR01008
 U 1 1 5F5D6E3D
 P 2350 6200
-F 0 "#PWR0111" H 2350 5950 50  0001 C CNN
+F 0 "#PWR01008" H 2350 5950 50  0001 C CNN
 F 1 "GND" H 2355 6027 50  0000 C CNN
 F 2 "" H 2350 6200 50  0001 C CNN
@@
 $EndComp
 $Comp
-L power:GNDA #PWR0112
+L power:GNDA #PWR01004
 U 1 1 5F5D7044
 P 1650 6200
-F 0 "#PWR0112" H 1650 5950 50  0001 C CNN
+F 0 "#PWR01004" H 1650 5950 50  0001 C CNN
 F 1 "GNDA" H 1655 6027 50  0000 C CNN
 F 2 "" H 1650 6200 50  0001 C CNN
@@
 $EndComp
 $Comp
-L power:+5V #PWR0113
+L power:+5V #PWR01007
 U 1 1 5F5D7F99
 P 2350 5600
-F 0 "#PWR0113" H 2350 5450 50  0001 C CNN
+F 0 "#PWR01007" H 2350 5450 50  0001 C CNN
 F 1 "+5V" H 2365 5773 50  0000 C CNN
 F 2 "" H 2350 5600 50  0001 C CNN
@@
 $EndComp
 $Comp
-L power:+5V #PWR0114
+L power:+5V #PWR01003
 U 1 1 5F5D85DF
 P 1650 5600
-F 0 "#PWR0114" H 1650 5450 50  0001 C CNN
+F 0 "#PWR01003" H 1650 5450 50  0001 C CNN
 F 1 "+5V" H 1665 5773 50  0000 C CNN
 F 2 "" H 1650 5600 50  0001 C CNN
@@
 	1650 6200 1750 6200
 $Comp
-L power:+1V8 #PWR0115
+L power:+1V8 #PWR01011
 U 1 1 5F5D95A1
 P 5200 5650
-F 0 "#PWR0115" H 5200 5500 50  0001 C CNN
+F 0 "#PWR01011" H 5200 5500 50  0001 C CNN
 F 1 "+1V8" H 5215 5823 50  0000 C CNN
 F 2 "" H 5200 5650 50  0001 C CNN
@@
 $EndComp
 $Comp
-L power:+1V8 #PWR0116
+L power:+1V8 #PWR01015
 U 1 1 5F5D9DEB
 P 5900 5650
-F 0 "#PWR0116" H 5900 5500 50  0001 C CNN
+F 0 "#PWR01015" H 5900 5500 50  0001 C CNN
 F 1 "+1V8" H 5915 5823 50  0000 C CNN
 F 2 "" H 5900 5650 50  0001 C CNN
@@
 $EndComp
 $Comp
-L power:GND #PWR0117
+L power:GND #PWR01012
 U 1 1 5F5DA1E2
 P 5200 5950
-F 0 "#PWR0117" H 5200 5700 50  0001 C CNN
+F 0 "#PWR01012" H 5200 5700 50  0001 C CNN
 F 1 "GND" H 5205 5777 50  0000 C CNN
 F 2 "" H 5200 5950 50  0001 C CNN
@@
 $EndComp
 $Comp
-L power:GND #PWR0118
+L power:GND #PWR01016
 U 1 1 5F5DA623
 P 5900 5950
-F 0 "#PWR0118" H 5900 5700 50  0001 C CNN
+F 0 "#PWR01016" H 5900 5700 50  0001 C CNN
 F 1 "GND" H 5905 5777 50  0000 C CNN
 F 2 "" H 5900 5950 50  0001 C CNN
