File: Outside-com.sch (KiCad schematic (older format))
At the start: 0 parts

Commit message: More of the same
Signed-off-by: Eldalote <Eldalote.Electronics@gmail.com>
Parts:
- added J601, J602: Conn_02x10_Row_Letter_First, Connector_PinHeader_2.54mm:PinHeader_2x10_P2.54mm_Vertical, symbol Connector_Generic:Conn_02x10_Odd_Even
Changed lines of the file:
@@
 Comment4 ""
 $EndDescr
+$Comp
+L Connector_Generic:Conn_02x10_Odd_Even J601
+U 1 1 5F5BFD4F
+P 3150 1950
+F 0 "J601" H 3200 2567 50  0000 C CNN
+F 1 "Conn_02x10_Row_Letter_First" H 3200 2476 50  0000 C CNN
+F 2 "Connector_PinHeader_2.54mm:PinHeader_2x10_P2.54mm_Vertical" H 3150 1950 50  0001 C CNN
+F 3 "~" H 3150 1950 50  0001 C CNN
+	1    3150 1950
+	1    0    0    -1
+$EndComp
+$Comp
+L Connector_Generic:Conn_02x10_Odd_Even J602
+U 1 1 5F5C4649
+P 3200 3200
+F 0 "J602" H 3250 3817 50  0000 C CNN
+F 1 "Conn_02x10_Row_Letter_First" H 3250 3726 50  0000 C CNN
+F 2 "Connector_PinHeader_2.54mm:PinHeader_2x10_P2.54mm_Vertical" H 3200 3200 50  0001 C CNN
+F 3 "~" H 3200 3200 50  0001 C CNN
+	1    3200 3200
+	1    0    0    -1
+$EndComp
 $EndSCHEMATC

Commit message: Further work
Signed-off-by: Eldalote <Eldalote.Electronics@gmail.com>
Parts:
- removed J601, J602: Conn_02x10_Row_Letter_First, Connector_PinHeader_2.54mm:PinHeader_2x10_P2.54mm_Vertical, symbol Connector_Generic:Conn_02x10_Odd_Even
Changed lines of the file:
@@
 $Descr A4 11693 8268
 encoding utf-8
-Sheet 6 11
+Sheet 6 12
 Title ""
 Date ""
@@
 Comment4 ""
 $EndDescr
-$Comp
-L Connector_Generic:Conn_02x10_Odd_Even J601
-U 1 1 5F5BFD4F
-P 3150 1950
-F 0 "J601" H 3200 2567 50  0000 C CNN
-F 1 "Conn_02x10_Row_Letter_First" H 3200 2476 50  0000 C CNN
-F 2 "Connector_PinHeader_2.54mm:PinHeader_2x10_P2.54mm_Vertical" H 3150 1950 50  0001 C CNN
-F 3 "~" H 3150 1950 50  0001 C CNN
-	1    3150 1950
-	1    0    0    -1
-$EndComp
-$Comp
-L Connector_Generic:Conn_02x10_Odd_Even J602
-U 1 1 5F5C4649
-P 3200 3200
-F 0 "J602" H 3250 3817 50  0000 C CNN
-F 1 "Conn_02x10_Row_Letter_First" H 3250 3726 50  0000 C CNN
-F 2 "Connector_PinHeader_2.54mm:PinHeader_2x10_P2.54mm_Vertical" H 3200 3200 50  0001 C CNN
-F 3 "~" H 3200 3200 50  0001 C CNN
-	1    3200 3200
-	1    0    0    -1
-$EndComp
+$Sheet
+S 4900 1900 1750 1300
+U 5F5C1DDB
+F0 "GPIOs" 50
+F1 "GPIO.sch" 50
+$EndSheet
 $EndSCHEMATC
