File: nRF24L01p-radio.sch (KiCad schematic (older format))
At the start: 31 parts, among them J501 SMA-RP, U501 nRF24L01P, U502 RFX2401C, X501 16MHz

Commit message: Started PCB layout planning
Signed-off-by: Eldalote <Eldalote.Electronics@gmail.com>
Parts:
- removed LOGO501: Logo_Open_Hardware_Small, Symbol:OSHW-Logo2_7.3x6mm_SilkScreen, symbol Graphic:Logo_Open_Hardware_Small
- removed X501: 16MHz, Crystal:Crystal_SMD_3225-4Pin_3.2x2.5mm, symbol Device:Crystal
- added X501: 16MHz, Crystal:Crystal_SMD_3225-4Pin_3.2x2.5mm, symbol Device:Crystal_GND24_Small
Connections:
- wire segments 119 -> 125
Other:
- note removed: "Copyright (C) 2020 J.M. Liewes\n\nThis documentation describes Open Hardware and is licensed under the CERN OHL v. 1.2\n\n.You may redistribute and modify this documentation under the terms of the CERN OHL v.1.2. (http://ohwr.org/cernohl). \nThis documentation is distributed WITHOUT ANY EXPRESS OR IMPLIED WARRANTY, INCLUDING OF MERCHANTABILITY, \nSATISFACTORY QUALITY AND FITNESS FOR A PARTICULAR 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"
Changed lines of the file:
@@
 $Descr A4 11693 8268
 encoding utf-8
-Sheet 5 7
+Sheet 5 11
 Title ""
 Date ""
@@
 	1    0    0    -1
 $EndComp
-$Comp
-L Device:Crystal X501
-U 1 1 5F3B34D3
-P 3250 4350
-F 0 "X501" H 3250 4500 50  0000 C CNN
-F 1 "16MHz" H 3250 4200 50  0000 C CNN
-F 2 "Crystal:Crystal_SMD_3225-4Pin_3.2x2.5mm" H 3250 4350 50  0001 C CNN
-F 3 "https://datasheet.lcsc.com/szlcsc/Yangxing-Tech-X322516MLB4SI_C13738.pdf" H 3250 4350 50  0001 C CNN
-F 4 "" V 3250 4350 50  0001 C CNN "JLC Part Nr"
-F 5 " C13738" H 3250 4350 50  0001 C CNN "LCSC"
-	1    3250 4350
-	1    0    0    -1
-$EndComp
 Wire Wire Line
 	2800 3950 3100 3950
@@
 	0    -1   -1   0
 $EndComp
-Connection ~ 3100 4350
-Connection ~ 3400 4350
 Wire Wire Line
 	2800 3150 3050 3150
@@
 Wire Wire Line
 	4600 2700 4600 3150
-Wire Wire Line
-	3450 3150 4600 3150
 Wire Wire Line
 	3250 2700 3250 2950
@@
 Wire Wire Line
 	5700 2500 5700 2400
-Wire Wire Line
-	5200 2400 5200 3000
 $Comp
 L power:GND #PWR0513
@@
 	1    5550 4450
 	0    -1   -1   0
-$EndComp
-$Comp
-L SamacSys_Parts:RFX2401C U502
-U 1 1 5F36A433
-P 5300 3200
-F 0 "U502" H 6350 3700 50  0000 L CNN
-F 1 "RFX2401C" H 6350 3600 50  0000 L CNN
-F 2 "QFN50P300X300X60-17N-D" H 6350 3700 50  0001 L CNN
-F 3 "http://www.skyworksinc.com/uploads/documents/RFX2401C_204359A.pdf" H 6350 3600 50  0001 L CNN
-F 4 "RF Front End 2.4GHz ZigBee/ISM RFeIC PA+LNA+SPDT" H 6350 3500 50  0001 L CNN "Description"
-F 5 "0.6" H 6350 3400 50  0001 L CNN "Height"
-F 6 "477-RFX2401C" H 6350 3300 50  0001 L CNN "Mouser Part Number"
-F 7 "https://www.mouser.co.uk/ProductDetail/Skyworks-Solutions-Inc/RFX2401C?qs=dBWc1juS%252B3ydEXrKsuxQ7A%3D%3D" H 6350 3200 50  0001 L CNN "Mouser Price/Stock"
-F 8 "Skyworks" H 6350 3100 50  0001 L CNN "Manufacturer_Name"
-F 9 "RFX2401C" H 6350 3000 50  0001 L CNN "Manufacturer_Part_Number"
-F 10 " C19213" H 5300 3200 50  0001 C CNN "LCSC"
-F 11 "863-1828-1-ND " H 5300 3200 50  0001 C CNN "DigiKey"
-F 12 "477-RFX2401C " H 5300 3200 50  0001 C CNN "Mouser"
-	1    5300 3200
-	1    0    0    -1
 $EndComp
 $Comp
@@
 Wire Wire Line
 	5800 4700 5800 4750
-Text Notes 7000 7100 0    34   ~ 0
-Copyright (C) 2020 J.M. Liewes\n\nThis documentation describes Open Hardware and is licensed under the CERN OHL v. 1.2\n\n.You may redistribute and modify this documentation under the terms of the CERN OHL v.1.2. (http://ohwr.org/cernohl). \nThis documentation is distributed WITHOUT ANY EXPRESS OR IMPLIED WARRANTY, INCLUDING OF MERCHANTABILITY, \nSATISFACTORY QUALITY AND FITNESS FOR A PARTICULAR PURPOSE.  Please see the CERN OHL v.1.2 for applicable conditions\n\nIf you chose to manufacture products based on this design, please notify me (see license section 4.2) via Eldalote.Electronics@gmail.com
-$Comp
-L Graphic:Logo_Open_Hardware_Small LOGO501
-U 1 1 5F43547C
-P 10950 6900
-F 0 "LOGO501" H 10950 7175 50  0001 C CNN
-F 1 "Logo_Open_Hardware_Small" H 10950 6675 50  0001 C CNN
-F 2 "Symbol:OSHW-Logo2_7.3x6mm_SilkScreen" H 10950 6900 50  0001 C CNN
-F 3 "~" H 10950 6900 50  0001 C CNN
-	1    10950 6900
-	1    0    0    -1
-$EndComp
 $Comp
 L RF:nRF24L01P U501
@@
 Text Notes 8200 4700 0    118  ~ 0
 InOut ports\n
+Wire Wire Line
+	5200 2400 5200 3000
+Wire Wire Line
+	3450 3150 4600 3150
+$Comp
+L SamacSys_Parts:RFX2401C U502
+U 1 1 5F36A433
+P 5300 3200
+F 0 "U502" H 6350 3700 50  0000 L CNN
+F 1 "RFX2401C" H 6350 3600 50  0000 L CNN
+F 2 "QFN50P300X300X60-17N-D" H 6350 3700 50  0001 L CNN
+F 3 "http://www.skyworksinc.com/uploads/documents/RFX2401C_204359A.pdf" H 6350 3600 50  0001 L CNN
+F 4 "RF Front End 2.4GHz ZigBee/ISM RFeIC PA+LNA+SPDT" H 6350 3500 50  0001 L CNN "Description"
+F 5 "0.6" H 6350 3400 50  0001 L CNN "Height"
+F 6 "477-RFX2401C" H 6350 3300 50  0001 L CNN "Mouser Part Number"
+F 7 "https://www.mouser.co.uk/ProductDetail/Skyworks-Solutions-Inc/RFX2401C?qs=dBWc1juS%252B3ydEXrKsuxQ7A%3D%3D" H 6350 3200 50  0001 L CNN "Mouser Price/Stock"
+F 8 "Skyworks" H 6350 3100 50  0001 L CNN "Manufacturer_Name"
+F 9 "RFX2401C" H 6350 3000 50  0001 L CNN "Manufacturer_Part_Number"
+F 10 " C19213" H 5300 3200 50  0001 C CNN "LCSC"
+F 11 "863-1828-1-ND " H 5300 3200 50  0001 C CNN "DigiKey"
+F 12 "477-RFX2401C " H 5300 3200 50  0001 C CNN "Mouser"
+	1    5300 3200
+	1    0    0    -1
+$EndComp
+$Comp
+L Device:Crystal_GND24_Small X501
+U 1 1 5F60AD74
+P 3250 4350
+F 0 "X501" H 3550 4400 50  0000 L CNN
+F 1 "16MHz" H 3500 4300 50  0000 L CNN
+F 2 "Crystal:Crystal_SMD_3225-4Pin_3.2x2.5mm" H 3250 4350 50  0001 C CNN
+F 3 "~" H 3250 4350 50  0001 C CNN
+	1    3250 4350
+	1    0    0    -1
+$EndComp
+Wire Wire Line
+	3400 4350 3350 4350
+Connection ~ 3400 4350
+Wire Wire Line
+	3100 4350 3150 4350
+Connection ~ 3100 4350
+$Comp
+L power:GND #PWR?
+U 1 1 5F615159
+P 3250 4500
+F 0 "#PWR?" H 3250 4250 50  0001 C CNN
+F 1 "GND" H 3255 4327 50  0000 C CNN
+F 2 "" H 3250 4500 50  0001 C CNN
+F 3 "" H 3250 4500 50  0001 C CNN
+	1    3250 4500
+	1    0    0    -1
+$EndComp
+$Comp
+L power:GND #PWR?
+U 1 1 5F6155A3
+P 3350 4000
+F 0 "#PWR?" H 3350 3750 50  0001 C CNN
+F 1 "GND" H 3355 3827 50  0000 C CNN
+F 2 "" H 3350 4000 50  0001 C CNN
+F 3 "" H 3350 4000 50  0001 C CNN
+	1    3350 4000
+	1    0    0    -1
+$EndComp
+Wire Wire Line
+	3250 4450 3250 4500
+Wire Wire Line
+	3250 4250 3250 3950
+Wire Wire Line
+	3250 3950 3350 3950
+Wire Wire Line
+	3350 3950 3350 4000
 $EndSCHEMATC

Commit message: Made progress woth power
Signed-off-by: Jan Mart Liewes <Eldalote.Electronics@gmail.com>
Parts:
- removed C505: 22pF, Capacitor_SMD:C_0402_1005Metric, symbol Device:C_Small
- added C805: 15pF, Capacitor_SMD:C_0402_1005Metric, symbol Device:C_Small
- C804: renamed from C504; value 22pF -> 15pF; LCSC C1555 -> C1548
- renumbered C501 to C801, C502 to C802, C503 to C803, C506 to C806, C507 to C807, C508 to C808, C509 to C809, C510 to C810, C511 to C811, C512 to C812, C513 to C813, C514 to C814, C515 to C815, C516 to C816, C517 to C817, J501 to J801, L501 to L801, L502 to L802, L503 to L803, L504 to L804, L505 to L805, R501 to R801, R502 to R802, R503 to R803, R504 to R804, U501 to U801, U502 to U802, X501 to X801
