File: 5v-power-regulator.sch (KiCad schematic (older format))
At the start: 6 parts, among them U301 AP63205WU-7

Commit message: Finished v0.1 of power, and v0.1 of sensors.
Signed-off-by: Jan Mart Liewes <Eldalote.Electronics@gmail.com>
Parts:
- L301: value 4.7uH 2.6ADC -> 4u7H 2.6ADC
Changed lines of the file:
@@
 P 5900 3450
 F 0 "L301" V 6090 3450 50  0000 C CNN
-F 1 "4.7uH 2.6ADC" V 5999 3450 50  0000 C CNN
+F 1 "4u7H 2.6ADC" V 5999 3450 50  0000 C CNN
 F 2 "Eldalote-footprints:L_5030_TAIYO_YUDEN" H 5900 3450 50  0001 C CNN
 F 3 "~" H 5900 3450 50  0001 C CNN
