File: Sensors.sch (KiCad schematic (older format))
At the start: 5 parts, among them U401 ICM-20948, U402 BNO055, U403 DPS422XTSA1, U404 MCP3208

Commit message: Started PCB layout planning
Signed-off-by: Eldalote <Eldalote.Electronics@gmail.com>
Parts:
- gave numbers to parts that had none: 1
Changed lines of the file:
@@
 $Descr A4 11693 8268
 encoding utf-8
-Sheet 4 7
+Sheet 4 11
 Title ""
 Date ""
@@
 $EndComp
 $Comp
-L dk_Logic-Translators-Level-Shifters:TXB0104PWR U?
+L dk_Logic-Translators-Level-Shifters:TXB0104PWR U405
 U 1 1 5F4C621A
 P 10150 5000
-F 0 "U?" H 10100 4403 60  0000 C CNN
+F 0 "U405" H 10100 4403 60  0000 C CNN
 F 1 "TXB0104PWR" H 10100 4297 60  0000 C CNN
 F 2 "digikey-footprints:TSSOP-14_W4.4mm" H 10350 5200 60  0001 L CNN

Commit message: More of the same
Signed-off-by: Eldalote <Eldalote.Electronics@gmail.com>
Parts:
- removed U405: TXB0104PWR, digikey-footprints:TSSOP-14_W4.4mm, symbol dk_Logic-Translators-Level-Shifters:TXB0104PWR
- added U405, U406: TXB0108PWR, digikey-footprints:TSSOP-20_W4.4mm, symbol dk_Logic-Translators-Level-Shifters:TXB0108PWR
Changed lines of the file:
@@
 $EndComp
 $Comp
-L dk_Logic-Translators-Level-Shifters:TXB0104PWR U405
-U 1 1 5F4C621A
-P 10150 5000
-F 0 "U405" H 10100 4403 60  0000 C CNN
-F 1 "TXB0104PWR" H 10100 4297 60  0000 C CNN
-F 2 "digikey-footprints:TSSOP-14_W4.4mm" H 10350 5200 60  0001 L CNN
-F 3 "http://www.ti.com/general/docs/suppproductinfo.tsp?distId=10&gotoUrl=http%3A%2F%2Fwww.ti.com%2Flit%2Fgpn%2Ftxb0104" H 10350 5300 60  0001 L CNN
-F 4 "296-21929-1-ND" H 10350 5400 60  0001 L CNN "Digi-Key_PN"
-F 5 "TXB0104PWR" H 10350 5500 60  0001 L CNN "MPN"
-F 6 "Integrated Circuits (ICs)" H 10350 5600 60  0001 L CNN "Category"
-F 7 "Logic - Translators, Level Shifters" H 10350 5700 60  0001 L CNN "Family"
-F 8 "http://www.ti.com/general/docs/suppproductinfo.tsp?distId=10&gotoUrl=http%3A%2F%2Fwww.ti.com%2Flit%2Fgpn%2Ftxb0104" H 10350 5800 60  0001 L CNN "DK_Datasheet_Link"
-F 9 "/product-detail/en/texas-instruments/TXB0104PWR/296-21929-1-ND/1629282" H 10350 5900 60  0001 L CNN "DK_Detail_Page"
-F 10 "IC TRNSLTR BIDIRECTIONAL 14TSSOP" H 10350 6000 60  0001 L CNN "Description"
-F 11 "Texas Instruments" H 10350 6100 60  0001 L CNN "Manufacturer"
-F 12 "Active" H 10350 6200 60  0001 L CNN "Status"
-F 13 "296-21929-1-ND" H 10150 5000 50  0001 C CNN "DigiKey"
-F 14 "595-TXB0104PWR " H 10150 5000 50  0001 C CNN "Mouser"
-	1    10150 5000
+L dk_Logic-Translators-Level-Shifters:TXB0108PWR U406
+U 1 1 5F5EB69B
+P 10050 5200
+F 0 "U406" H 10000 4403 60  0000 C CNN
+F 1 "TXB0108PWR" H 10000 4297 60  0000 C CNN
+F 2 "digikey-footprints:TSSOP-20_W4.4mm" H 10250 5400 60  0001 L CNN
+F 3 "http://www.ti.com/general/docs/suppproductinfo.tsp?distId=10&gotoUrl=http%3A%2F%2Fwww.ti.com%2Flit%2Fgpn%2Ftxb0108" H 10250 5500 60  0001 L CNN
+F 4 "296-21527-1-ND" H 10250 5600 60  0001 L CNN "Digi-Key_PN"
+F 5 "TXB0108PWR" H 10250 5700 60  0001 L CNN "MPN"
+F 6 "Integrated Circuits (ICs)" H 10250 5800 60  0001 L CNN "Category"
+F 7 "Logic - Translators, Level Shifters" H 10250 5900 60  0001 L CNN "Family"
+F 8 "http://www.ti.com/general/docs/suppproductinfo.tsp?distId=10&gotoUrl=http%3A%2F%2Fwww.ti.com%2Flit%2Fgpn%2Ftxb0108" H 10250 6000 60  0001 L CNN "DK_Datasheet_Link"
+F 9 "/product-detail/en/texas-instruments/TXB0108PWR/296-21527-1-ND/1305700" H 10250 6100 60  0001 L CNN "DK_Detail_Page"
+F 10 "IC TRNSLTR BIDIRECTIONAL 20TSSOP" H 10250 6200 60  0001 L CNN "Description"
+F 11 "Texas Instruments" H 10250 6300 60  0001 L CNN "Manufacturer"
+F 12 "Active" H 10250 6400 60  0001 L CNN "Status"
+	1    10050 5200
 	1    0    0    -1
 $EndComp
+$Comp
+L dk_Logic-Translators-Level-Shifters:TXB0108PWR U405
+U 1 1 5F5F3BD5
+P 2000 3000
+F 0 "U405" H 1950 2203 60  0000 C CNN
+F 1 "TXB0108PWR" H 1950 2097 60  0000 C CNN
+F 2 "digikey-footprints:TSSOP-20_W4.4mm" H 2200 3200 60  0001 L CNN
+F 3 "http://www.ti.com/general/docs/suppproductinfo.tsp?distId=10&gotoUrl=http%3A%2F%2Fwww.ti.com%2Flit%2Fgpn%2Ftxb0108" H 2200 3300 60  0001 L CNN
+F 4 "296-21527-1-ND" H 2200 3400 60  0001 L CNN "Digi-Key_PN"
+F 5 "TXB0108PWR" H 2200 3500 60  0001 L CNN "MPN"
+F 6 "Integrated Circuits (ICs)" H 2200 3600 60  0001 L CNN "Category"
+F 7 "Logic - Translators, Level Shifters" H 2200 3700 60  0001 L CNN "Family"
+F 8 "http://www.ti.com/general/docs/suppproductinfo.tsp?distId=10&gotoUrl=http%3A%2F%2Fwww.ti.com%2Flit%2Fgpn%2Ftxb0108" H 2200 3800 60  0001 L CNN "DK_Datasheet_Link"
+F 9 "/product-detail/en/texas-instruments/TXB0108PWR/296-21527-1-ND/1305700" H 2200 3900 60  0001 L CNN "DK_Detail_Page"
+F 10 "IC TRNSLTR BIDIRECTIONAL 20TSSOP" H 2200 4000 60  0001 L CNN "Description"
+F 11 "Texas Instruments" H 2200 4100 60  0001 L CNN "Manufacturer"
+F 12 "Active" H 2200 4200 60  0001 L CNN "Status"
+	1    2000 3000
+	1    0    0    -1
+$EndComp

Commit message: Made progress woth power
Signed-off-by: Jan Mart Liewes <Eldalote.Electronics@gmail.com>
Parts:
- removed U401: ICM-20948, Sensor_Motion:InvenSense_QFN-24_3x3mm_P0.4mm, symbol Sensor_Motion:ICM-20948
- removed U405: TXB0108PWR, digikey-footprints:TSSOP-20_W4.4mm, symbol dk_Logic-Translators-Level-Shifters:TXB0108PWR
- renumbered U402 to U701, U403 to U702, U404 to U703, U406 to U704
Changed lines of the file:
@@
 $Descr A4 11693 8268
 encoding utf-8
-Sheet 4 12
+Sheet 4 15
 Title ""
 Date ""
@@
 $EndDescr
 $Comp
-L Sensor_Motion:ICM-20948 U401
-U 1 1 5F4BD0F1
-P 3850 3050
-F 0 "U401" H 3850 2261 50  0000 C CNN
-F 1 "ICM-20948" H 3850 2170 50  0000 C CNN
-F 2 "Sensor_Motion:InvenSense_QFN-24_3x3mm_P0.4mm" H 3850 2050 50  0001 C CNN
-F 3 "http://www.invensense.com/wp-content/uploads/2016/06/DS-000189-ICM-20948-v1.3.pdf" H 3850 2900 50  0001 C CNN
-F 4 "1428-1123-1-ND" H 3850 3050 50  0001 C CNN "DigiKey"
-F 5 "410-ICM-20948 " H 3850 3050 50  0001 C CNN "Mouser"
-	1    3850 3050
-	1    0    0    -1
-$EndComp
-$Comp
-L Sensor_Motion:BNO055 U402
+L Sensor_Motion:BNO055 U701
 U 1 1 5F4BD31D
 P 6350 3050
-F 0 "U402" H 6350 3931 50  0000 C CNN
+F 0 "U701" H 6350 3931 50  0000 C CNN
 F 1 "BNO055" H 6350 3840 50  0000 C CNN
 F 2 "Package_LGA:LGA-28_5.2x3.8mm_P0.5mm" H 6600 2400 50  0001 L CNN
@@
 $EndComp
 $Comp
-L 2020-08-24_12-35-16:DPS422XTSA1 U403
+L 2020-08-24_12-35-16:DPS422XTSA1 U702
 U 1 1 5F4C1DB6
 P 7850 2950
-F 0 "U403" H 8650 3337 60  0000 C CNN
+F 0 "U702" H 8650 3337 60  0000 C CNN
 F 1 "DPS422XTSA1" H 8650 3231 60  0000 C CNN
 F 2 "footprints:DPS422XTSA1" H 8650 3190 60  0001 C CNN
@@
 $EndComp
 $Comp
-L Analog_ADC:MCP3208 U404
+L Analog_ADC:MCP3208 U703
 U 1 1 5F4C395E
 P 8700 5000
-F 0 "U404" H 8700 5681 50  0000 C CNN
+F 0 "U703" H 8700 5681 50  0000 C CNN
 F 1 "MCP3208" H 8700 5590 50  0000 C CNN
 F 2 "Package_SO:SOIC-16_3.9x9.9mm_P1.27mm" H 8800 5100 50  0001 C CNN
@@
 $EndComp
 $Comp
-L dk_Logic-Translators-Level-Shifters:TXB0108PWR U406
+L dk_Logic-Translators-Level-Shifters:TXB0108PWR U704
 U 1 1 5F5EB69B
 P 10050 5200
-F 0 "U406" H 10000 4403 60  0000 C CNN
+F 0 "U704" H 10000 4403 60  0000 C CNN
 F 1 "TXB0108PWR" H 10000 4297 60  0000 C CNN
 F 2 "digikey-footprints:TSSOP-20_W4.4mm" H 10250 5400 60  0001 L CNN
@@
 	1    0    0    -1
 $EndComp
-$Comp
-L dk_Logic-Translators-Level-Shifters:TXB0108PWR U405
-U 1 1 5F5F3BD5
-P 2000 3000
-F 0 "U405" H 1950 2203 60  0000 C CNN
-F 1 "TXB0108PWR" H 1950 2097 60  0000 C CNN
-F 2 "digikey-footprints:TSSOP-20_W4.4mm" H 2200 3200 60  0001 L CNN
-F 3 "http://www.ti.com/general/docs/suppproductinfo.tsp?distId=10&gotoUrl=http%3A%2F%2Fwww.ti.com%2Flit%2Fgpn%2Ftxb0108" H 2200 3300 60  0001 L CNN
-F 4 "296-21527-1-ND" H 2200 3400 60  0001 L CNN "Digi-Key_PN"
-F 5 "TXB0108PWR" H 2200 3500 60  0001 L CNN "MPN"
-F 6 "Integrated Circuits (ICs)" H 2200 3600 60  0001 L CNN "Category"
-F 7 "Logic - Translators, Level Shifters" H 2200 3700 60  0001 L CNN "Family"
-F 8 "http://www.ti.com/general/docs/suppproductinfo.tsp?distId=10&gotoUrl=http%3A%2F%2Fwww.ti.com%2Flit%2Fgpn%2Ftxb0108" H 2200 3800 60  0001 L CNN "DK_Datasheet_Link"
-F 9 "/product-detail/en/texas-instruments/TXB0108PWR/296-21527-1-ND/1305700" H 2200 3900 60  0001 L CNN "DK_Detail_Page"
-F 10 "IC TRNSLTR BIDIRECTIONAL 20TSSOP" H 2200 4000 60  0001 L CNN "Description"
-F 11 "Texas Instruments" H 2200 4100 60  0001 L CNN "Manufacturer"
-F 12 "Active" H 2200 4200 60  0001 L CNN "Status"
-	1    2000 3000
-	1    0    0    -1
-$EndComp

Commit message: Finished v0.1 of power, and v0.1 of sensors.
Signed-off-by: Jan Mart Liewes <Eldalote.Electronics@gmail.com>
Parts:
- added C701, C703, C705, C708, C709, C713, C716: 100nF, Capacitor_SMD:C_0402_1005Metric, symbol Device:C_Small
- added C702: 2u2F, Capacitor_SMD:C_0603_1608Metric, symbol Device:C_Small
- added C704: 10nF, Capacitor_SMD:C_0402_1005Metric, symbol Device:C_Small
- added C706, C707, C715, C718: 100nF, Capacitor_SMD:C_0805_2012Metric_Pad1.15x1.40mm_HandSolder, symbol Device:C_Small
- added C710: 4n7F, Capacitor_SMD:C_0603_1608Metric, symbol Device:C_Small
- added C711, C712: 22pF, Capacitor_SMD:C_0603_1608Metric, symbol Device:C_Small
- added C714, C717: 1uF, Capacitor_SMD:C_0805_2012Metric_Pad1.15x1.40mm_HandSolder, symbol Device:C_Small
- added R701, R702: 4k7, Resistor_SMD:R_0402_1005Metric, symbol Device:R
- added R703: 10k, Resistor_SMD:R_0402_1005Metric, symbol Device:R
- added R704: 10K, Resistor_SMD:R_0805_2012Metric_Pad1.15x1.40mm_HandSolder, symbol Device:R
- added U701: ICM-20602, Package_LGA:LGA-16_3x3mm_P0.5mm_LayoutBorder3x5y, symbol Sensor_Motion:ICM-20602
- added Y701: 32.7KHz, Crystal:Crystal_SMD_3215-2Pin_3.2x1.5mm, symbol Device:Crystal
- renumbered U704 to U702, U701 to U703, U702 to U704, U703 to U705
Connections:
- net BNO_NRESET: now reaches U703.11 (~RESET)
- net BNO_NRESET: now also R703.2
- net BNO_INT: now reaches U703.14 (INT)
- net GND: now reaches U703.15 (GNDIO), U703.16 (GNDIO), U703.25 (GNDIO)
- net GND: now also U702.11 (GND), U703.17 (COM3), U703.18 (COM2), U703.2 (GND), U703.5 (PS1), U703.6 (PS0), U704.1 (GND), U704.7 (GND), U705.9 (DGND), C701.2, C702.2, C703.2, C704.2, C705.2, C706.2, C707.2, C708.2, C709.2, C710.2, C711.1, C712.1, C713.2, C714.2, C715.2, C716.2, C717.2, C718.2, R704.2, U701.10 (GND), U701.11 (GND), U701.12 (GND), U701.13 (GND), U701.15 (GND), U701.9 (GND)
- net BNO_SCL: now reaches U703.19 (COM1)
- net BNO_SCL: now also R701.2
- net BNO_SDA: now reaches U703.20 (COM0)
- net BNO_SDA: now also R702.2
- net at U703.26 (XOUT32): now also C711.2, Y701.1
- net at U703.27 (XIN32): now also C712.2, Y701.2
- net +3V3: now reaches U703.28 (VDDIO)
- net +3V3: now also U702.2 (VCCA), U703.3 (VDD), U703.4 (~BOOT_LOAD_PIN), U704.6 (VDDIO), U704.8 (VDD), C701.1, C702.1, C704.1, C705.1, C706.1, C708.1, C710.1, C713.1, C716.1, R701.1, R702.1, R703.1, U701.1 (VDDIO), U701.16 (VDD)
- net at U703.9 (CAP): now also C709.1
- net DPS_CSn: now reaches U704.2 (CSB)
- net DPS_MOSI: now reaches U704.3 (SDI)
- net DPS_SCLK: now reaches U704.4 (SCK)
- net DPS_MISO: now reaches U704.5 (SDO)
- net ADC_CH0: now reaches U705.1 (CH0)
- net 5v_ADC_CSn: now reaches U705.10 (~CS~/SHDN)
- net 5v_ADC_CSn: now also U702.20 (B1)
- net 5v_ADC_Din: now reaches U705.11 (Din)
- net 5v_ADC_Din: now also U702.18 (B2)
- net 5v_ADC_Dout: now reaches U705.12 (Dout)
- net 5v_ADC_Dout: now also U702.17 (B3)
- net 5v_ADC_CLK: now reaches U705.13 (CLK)
- net 5v_ADC_CLK: now also U702.16 (B4)
- net GNDA: now reaches U705.14 (AGND)
- net +5V: now reaches U705.15 (Vref)
- net +5V: now also U702.19 (VCCB), U705.16 (Vdd), C707.1, C714.1, C715.1, C717.1, C718.1
- net ADC_CH1: now reaches U705.2 (CH1)
- net ADC_CH2: now reaches U705.3 (CH2)
- net ADC_CH3: now reaches U705.4 (CH3)
- net ADC_CH4: now reaches U705.5 (CH4)
- net ADC_CH5: now reaches U705.6 (CH5)
- net ADC_CH6: now reaches U705.7 (CH6)
- net ADC_CH7: now reaches U705.8 (CH7)
- net ADC_CSn: now reaches U702.1 (A1)
- net at U702.10 (OE): now also R704.1
- net 5v_GPIO_5v_3: now reaches U702.12 (B8)
- net 5v_GPIO_5v_2: now reaches U702.13 (B7)
- net 5v_GPIO_5v_1: now reaches U702.14 (B6)
- net 5v_GPIO_5v_0: now reaches U702.15 (B5)
- net ADC_MOSI: now reaches U702.3 (A2)
- net ADC_MISO: now reaches U702.4 (A3)
- net ADC_SCLK: now reaches U702.5 (A4)
- net 5v_GPIO_0: now reaches U702.6 (A5)
- net 5v_GPIO_1: now reaches U702.7 (A6)
- net 5v_GPIO_2: now reaches U702.8 (A7)
- net 5v_GPIO_3: now reaches U702.9 (A8)
- new net: C703.1, U701.14 (REGOUT)
- new net ICM_CSn: U701.5 (~CS)
- new net ICM_FSYNC: U701.8 (FSYNC)
- new net ICM_INT: U701.6 (INT)
- new net ICM_MISO: U701.4 (SAO/SD0)
- new net ICM_MOSI: U701.3 (SDA/SDI)
- new net ICM_SCLK: U701.2 (SCL/SPC)
- no-connect marks 0 -> 1
Other:
- note added: "5v-3v3 level translator"
- note added: "ADC"
- note added: "BNO 055"
- note added: "DPS422"
- note added: "ICM 20602"
- note added: "Sheet IO"
- moved on the sheet: U702, U703, U704, U705
